File: CatLasers.kicad_sch (KiCad schematic)
At the start: 9 parts, among them J2 Programmer, J3 Conn_01x04, J4 IR Emitter, J5 Conn_01x20, J6 Conn_01x04, J7 Power Jumper, U2 ESP32-WROOM-32E_(4MB_HIGH_TEM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

Commit message: Moved IR Emitter and Receiver to separate sheet
Parts:
- removed J4: IR Emitter, Connector_PinHeader_2.54mm:PinHeader_1x02_P2.54mm_Vertical, symbol Connector_Generic:Conn_01x02
- removed J6: Conn_01x04, Connector_PinHeader_2.54mm:PinHeader_1x04_P2.54mm_Vertical, symbol Connector_Generic:Conn_01x04
- removed MOSFET1: SSM3J328R, SOT-23F_TOS, symbol ProjPMOS_LV:SSM3J328R
- removed R8: R, Resistor_SMD:R_0805_2012Metric, symbol Hestres_Standard_Lib:R
Other:
- added sheet IR Emitter + Receiver (IR_EandR.kicad_sch)
Changed lines of the file:
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@@
   (junction (at 108.585 55.88) (diameter 0) (color 0 0 0 0)
   )
-  (junction (at 179.705 101.6) (diameter 0) (color 0 0 0 0)
-  )
   (junction (at 103.505 42.545) (diameter 0) (color 0 0 0 0)
   )
@@
     (stroke (width 0) (type default))
   )
-  (wire (pts (xy 179.705 100.33) (xy 179.705 101.6))
-    (stroke (width 0) (type default))
-  )
-  (wire (pts (xy 154.94 99.06) (xy 157.48 99.06))
-    (stroke (width 0) (type default))
-  )
   (wire (pts (xy 74.93 49.53) (xy 74.93 45.72))
     (stroke (width 0) (type default))
@@
     (stroke (width 0) (type default))
   )
-  (wire (pts (xy 179.705 101.6) (xy 179.705 104.775))
-    (stroke (width 0) (type default))
-  )
   (wire (pts (xy 109.22 109.22) (xy 105.41 109.22))
     (stroke (width 0) (type default))
@@
     (stroke (width 0) (type default))
   )
-  (wire (pts (xy 154.94 101.6) (xy 179.705 101.6))
-    (stroke (width 0) (type default))
-  )
   (wire (pts (xy 45.72 116.205) (xy 33.02 116.205))
     (stroke (width 0) (type default))
@@
     (stroke (width 0) (type default))
   )
-  (wire (pts (xy 157.48 99.06) (xy 157.48 90.17))
-    (stroke (width 0) (type default))
-  )
   (wire (pts (xy 74.93 49.53) (xy 76.835 49.53))
     (stroke (width 0) (type default))
@@
     (stroke (width 0) (type default))
   )
-  (wire (pts (xy 157.48 90.17) (xy 167.005 90.17))
-    (stroke (width 0) (type default))
-  )
   (wire (pts (xy 48.26 118.745) (xy 33.02 118.745))
     (stroke (width 0) (type default))
   )
   (wire (pts (xy 48.26 83.82) (xy 48.26 118.745))
-    (stroke (width 0) (type default))
-  )
-  (wire (pts (xy 179.705 107.315) (xy 179.705 111.76))
     (stroke (width 0) (type default))
   )
@@
     (property "Intersheetrefs" "${INTERSHEET_REFS}" (at 80.645 35.4172 90)
       (effects (font (size 1.27 1.27)) (justify left) hide)
-    )
-  )
-  (global_label "3.3V" (shape input) (at 179.705 80.01 90) (fields_autoplaced)
-    (effects (font (size 1.27 1.27)) (justify left))
-    (property "Intersheetrefs" "${INTERSHEET_REFS}" (at 179.705 72.9124 90)
-      (effects (font (size 1.27 1.27)) (justify left) hide)
-    )
-  )
-  (global_label "GND" (shape input) (at 179.705 119.38 270) (fields_autoplaced)
-    (effects (font (size 1.27 1.27)) (justify right))
-    (property "Intersheetrefs" "${INTERSHEET_REFS}" (at 179.705 126.2357 90)
-      (effects (font (size 1.27 1.27)) (justify right) hide)
     )
   )
@@
         (path "/b94f5b10-ee0c-4425-b025-e3a8bb3cc7b0"
           (reference "J5") (unit 1)
-        )
-      )
-    )
-  )
-  (symbol (lib_id "Hestres_Standard_Lib:R") (at 179.705 115.57 0) (unit 1)
-    (in_bom yes) (on_board yes) (dnp no) (fields_autoplaced)
-    (property "Reference" "R8" (at 181.61 114.3 0)
-      (effects (font (size 1.27 1.27)) (justify left))
-    )
-    (property "Value" "R" (at 181.61 116.84 0)
-      (effects (font (size 1.27 1.27)) (justify left))
-    )
-    (property "Footprint" "Resistor_SMD:R_0805_2012Metric" (at 177.927 115.57 90)
-      (effects (font (size 1.27 1.27)) hide)
-    )
-    (property "Datasheet" "~" (at 179.705 115.57 0)
-      (effects (font (size 1.27 1.27)) hide)
-    )
-    (pin "1")
-    (pin "2")
-    (instances
-      (project "CatLasers"
-        (path "/b94f5b10-ee0c-4425-b025-e3a8bb3cc7b0"
-          (reference "R8") (unit 1)
-        )
-      )
-    )
-  )
-  (symbol (lib_id "ProjPMOS_LV:SSM3J328R") (at 169.545 82.55 0) (unit 1)
-    (in_bom yes) (on_board yes) (dnp no) (fields_autoplaced)
-    (property "Reference" "MOSFET1" (at 184.785 88.9 0)
-      (effects (font (size 1.524 1.524)) (justify left))
-    )
-    (property "Value" "SSM3J328R" (at 184.785 91.44 0)
-      (effects (font (size 1.524 1.524)) (justify left))
-    )
-    (property "Footprint" "SOT-23F_TOS" (at 169.545 82.55 0)
-      (effects (font (size 1.27 1.27) italic) hide)
-    )
-    (property "Datasheet" "SSM3J328R" (at 169.545 82.55 0)
-      (effects (font (size 1.27 1.27) italic) hide)
-    )
-    (pin "1")
-    (pin "2")
-    (pin "3")
-    (instances
-      (project "CatLasers"
-        (path "/b94f5b10-ee0c-4425-b025-e3a8bb3cc7b0"
-          (reference "MOSFET1") (unit 1)
         )
       )
@@
     )
   )
-  (symbol (lib_id "Connector_Generic:Conn_01x04") (at 149.86 104.14 180) (unit 1)
-    (in_bom yes) (on_board yes) (dnp no) (fields_autoplaced)
-    (property "Reference" "J6" (at 149.86 93.345 0)
-      (effects (font (size 1.27 1.27)))
-    )
-    (property "Value" "Conn_01x04" (at 149.86 95.885 0)
-      (effects (font (size 1.27 1.27)))
-    )
-    (property "Footprint" "Connector_PinHeader_2.54mm:PinHeader_1x04_P2.54mm_Vertical" (at 149.86 104.14 0)
-      (effects (font (size 1.27 1.27)) hide)
-    )
-    (property "Datasheet" "~" (at 149.86 104.14 0)
-      (effects (font (size 1.27 1.27)) hide)
-    )
-    (pin "1")
-    (pin "2")
-    (pin "3")
-    (pin "4")
-    (instances
-      (project "CatLasers"
-        (path "/b94f5b10-ee0c-4425-b025-e3a8bb3cc7b0"
-          (reference "J6") (unit 1)
-        )
-      )
-    )
-  )
-  (symbol (lib_id "Connector_Generic:Conn_01x02") (at 184.785 104.775 0) (unit 1)
-    (in_bom yes) (on_board yes) (dnp no) (fields_autoplaced)
-    (property "Reference" "J4" (at 187.96 104.775 0)
-      (effects (font (size 1.27 1.27)) (justify left))
-    )
-    (property "Value" "IR Emitter" (at 187.96 107.315 0)
-      (effects (font (size 1.27 1.27)) (justify left))
-    )
-    (property "Footprint" "Connector_PinHeader_2.54mm:PinHeader_1x02_P2.54mm_Vertical" (at 184.785 104.775 0)
-      (effects (font (size 1.27 1.27)) hide)
-    )
-    (property "Datasheet" "~" (at 184.785 104.775 0)
-      (effects (font (size 1.27 1.27)) hide)
-    )
-    (pin "1")
-    (pin "2")
-    (instances
-      (project "CatLasers"
-        (path "/b94f5b10-ee0c-4425-b025-e3a8bb3cc7b0"
-          (reference "J4") (unit 1)
-        )
-      )
-    )
-  )
   (symbol (lib_id "Connector_Generic:Conn_01x04") (at 57.15 111.76 180) (unit 1)
     (in_bom yes) (on_board yes) (dnp no) (fields_autoplaced)
@@
       )
     )
+  )
+  (sheet (at 159.385 87.63) (size 37.465 29.21) (fields_autoplaced)
+    (stroke (width 0.1524) (type solid))
+    (fill (color 0 0 0 0.0000))
+    (property "Sheetname" "IR Emitter + Receiver" (at 159.385 86.9184 0)
+      (effects (font (size 1.27 1.27)) (justify left bottom))
+    )
+    (property "Sheetfile" "IR_EandR.kicad_sch" (at 159.385 117.4246 0)
+      (effects (font (size 1.27 1.27)) (justify left top))
+    )
+    (instances
+      (project "CatLasers"
+        (path "/b94f5b10-ee0c-4425-b025-e3a8bb3cc7b0" (page "4"))
+      )
+    )

Commit message: IR Receiver and Comparator
Connections:
- net IR Emitter + Receiver/Receiver: now reaches J5.20 (Pin_20)
Other:
- sheet IR Emitter + Receiver ports: added Emitter, Receiver; removed none
Changed lines of the file:
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@@
+    (stroke (width 0) (type default))
+  )
+  (wire (pts (xy 159.385 109.855) (xy 139.065 109.855))
     (stroke (width 0) (type default))
   )
@@
     (stroke (width 0) (type default))
   )
+  (wire (pts (xy 139.065 154.305) (xy 109.22 154.305))
+    (stroke (width 0) (type default))
+  )
   (wire (pts (xy 109.22 134.62) (xy 105.41 134.62))
     (stroke (width 0) (type default))
@@
     (stroke (width 0) (type default))
   )
+  (wire (pts (xy 109.22 154.305) (xy 109.22 149.86))
+    (stroke (width 0) (type default))
+  )
   (wire (pts (xy 74.93 49.53) (xy 76.835 49.53))
     (stroke (width 0) (type default))
@@
   )
   (wire (pts (xy 109.22 104.14) (xy 105.41 104.14))
+    (stroke (width 0) (type default))
+  )
+  (wire (pts (xy 139.065 109.855) (xy 139.065 154.305))
     (stroke (width 0) (type default))
   )
@@
       (effects (font (size 1.27 1.27)) (justify left top))
     )
-    (instances
+    (pin "Emitter" input (at 159.385 98.425 180)
+      (effects (font (size 1.27 1.27)) (justify left))
+    )
+    (pin "Receiver" input (at 159.385 109.855 180)
+      (effects (font (size 1.27 1.27)) (justify left))
+    )
+    (instances

Commit message: Annotations
Other:
- note added: "All IO pins from the MCU are sent to jumper pins. This is for the test board, as I'm unfamiliar with the ESP32 chip. In the 2 weeks while I wait for the pcb to arrive, I can write my program for the MCU without worrying that I'll have pins connected wrong."
- note added: "I'm using the CAPUF ESP32 Programmer. This pinout allows me to directly connect the programmer."
- moved on the sheet: J2
Changed lines of the file:
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@@
     (stroke (width 0) (type default))
   )
-  (wire (pts (xy 43.18 111.125) (xy 33.02 111.125))
+  (wire (pts (xy 43.18 115.57) (xy 33.02 115.57))
     (stroke (width 0) (type default))
   )
@@
     (stroke (width 0) (type default))
   )
-  (wire (pts (xy 43.18 127) (xy 43.18 111.125))
+  (wire (pts (xy 43.18 127) (xy 43.18 115.57))
     (stroke (width 0) (type default))
   )
@@
     (stroke (width 0) (type default))
   )
-  (wire (pts (xy 40.64 129.54) (xy 40.64 108.585))
+  (wire (pts (xy 40.64 129.54) (xy 40.64 113.03))
     (stroke (width 0) (type default))
   )
@@
     (stroke (width 0) (type default))
   )
-  (wire (pts (xy 45.72 99.06) (xy 45.72 116.205))
+  (wire (pts (xy 45.72 99.06) (xy 45.72 120.65))
     (stroke (width 0) (type default))
   )
@@
     (stroke (width 0) (type default))
   )
-  (wire (pts (xy 45.72 116.205) (xy 33.02 116.205))
+  (wire (pts (xy 45.72 120.65) (xy 33.02 120.65))
     (stroke (width 0) (type default))
   )
@@
     (stroke (width 0) (type default))
   )
-  (wire (pts (xy 48.26 118.745) (xy 33.02 118.745))
-    (stroke (width 0) (type default))
-  )
-  (wire (pts (xy 48.26 83.82) (xy 48.26 118.745))
+  (wire (pts (xy 48.26 123.19) (xy 33.02 123.19))
+    (stroke (width 0) (type default))
+  )
+  (wire (pts (xy 48.26 83.82) (xy 48.26 123.19))
     (stroke (width 0) (type default))
   )
@@
     (stroke (width 0) (type default))
   )
-  (wire (pts (xy 40.64 108.585) (xy 33.02 108.585))
+  (wire (pts (xy 40.64 113.03) (xy 33.02 113.03))
     (stroke (width 0) (type default))
   )
@@
     (stroke (width 0) (type default))
   )
-  (global_label "GND" (shape input) (at 33.02 113.665 0) (fields_autoplaced)
+  (text "I'm using the CAPUF ESP32 Programmer.\nThis pinout allows me to directly\nconnect the programmer."
+    (at 14.605 137.16 0)
+    (effects (font (size 1.27 1.27)) (justify left bottom))
+  )
+  (text "All IO pins from the MCU are sent to jumper pins.\nThis is for the test board, as I'm unfamiliar with the\nESP32 chip. In the 2 weeks while I wait for the pcb to\narrive, I can write my program for the MCU without\nworrying that I'll have pins connected wrong."
+    (at 77.47 168.275 0)
+    (effects (font (size 1.27 1.27)) (justify left bottom))
+  )
+  (global_label "GND" (shape input) (at 33.02 118.11 0) (fields_autoplaced)
     (effects (font (size 1.27 1.27)) (justify left))
-    (property "Intersheetrefs" "${INTERSHEET_REFS}" (at 39.8757 113.665 0)
+    (property "Intersheetrefs" "${INTERSHEET_REFS}" (at 39.8757 118.11 0)
       (effects (font (size 1.27 1.27)) (justify left) hide)
     )
@@
     )
   )
-  (global_label "3.3V" (shape input) (at 33.02 106.045 0) (fields_autoplaced)
+  (global_label "3.3V" (shape input) (at 33.02 110.49 0) (fields_autoplaced)
     (effects (font (size 1.27 1.27)) (justify left))
-    (property "Intersheetrefs" "${INTERSHEET_REFS}" (at 40.1176 106.045 0)
+    (property "Intersheetrefs" "${INTERSHEET_REFS}" (at 40.1176 110.49 0)
       (effects (font (size 1.27 1.27)) (justify left) hide)
     )
@@
     )
   )
-  (symbol (lib_id "Connector_Generic:Conn_01x08") (at 27.94 113.665 0) (mirror y) (unit 1)
+  (symbol (lib_id "Connector_Generic:Conn_01x08") (at 27.94 118.11 0) (mirror y) (unit 1)
     (in_bom yes) (on_board yes) (dnp no) (fields_autoplaced)
-    (property "Reference" "J2" (at 27.94 99.695 0)
-      (effects (font (size 1.27 1.27)))
-    )
-    (property "Value" "Programmer" (at 27.94 102.235 0)
-      (effects (font (size 1.27 1.27)))
-    )
-    (property "Footprint" "Connector_PinHeader_2.54mm:PinHeader_1x08_P2.54mm_Vertical" (at 27.94 113.665 0)
-      (effects (font (size 1.27 1.27)) hide)
-    )
-    (property "Datasheet" "~" (at 27.94 113.665 0)
-      (effects (font (size 1.27 1.27)) hide)
-    )
+    (property "Reference" "J2" (at 27.94 104.14 0)
+      (effects (font (size 1.27 1.27)))
+    )
+    (property "Value" "Programmer" (at 27.94 106.68 0)
+      (effects (font (size 1.27 1.27)))
+    )
+    (property "Footprint" "Connector_PinHeader_2.54mm:PinHeader_1x08_P2.54mm_Vertical" (at 27.94 118.11 0)
+      (effects (font (size 1.27 1.27)) hide)
+    )
+    (property "Datasheet" "~" (at 27.94 118.11 0)
+      (effects (font (size 1.27 1.27)) hide)
+    )
