File: CatLasers.kicad_sch (KiCad schematic)
At the start: 6 parts, among them J2 Programmer, J3 Conn_01x04, J5 Conn_01x20, J7 Power Jumper, J9 Conn_01x04, U2 ESP32-WROOM-32E_(4MB_HIGH_TEM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

Commit message: Emitter, Receiver, and board outline
Connections:
- net GND: now also J5.20 (Pin_20)
Changed lines of the file:
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@@
+    )
+  )
+  (global_label "GND" (shape input) (at 109.22 149.86 270) (fields_autoplaced)
+    (effects (font (size 1.27 1.27)) (justify right))
+    (property "Intersheetrefs" "${INTERSHEET_REFS}" (at 109.22 156.7157 90)
+      (effects (font (size 1.27 1.27)) (justify right) hide)
     )
   )

Commit message: DRC Pass
Connections:
- net GND: no longer U2.39_10 (GND), U2.39_11 (GND), U2.39_12 (GND), U2.39_13 (GND), U2.39_14 (GND), U2.39_15 (GND), U2.39_16 (GND), U2.39_17 (GND), U2.39_18 (GND), U2.39_19 (GND), U2.39_20 (GND), U2.39_21 (GND)
Changed lines of the file:
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@@
     (pin "8")
     (pin "9")
-    (pin "39_10")
-    (pin "39_11")
-    (pin "39_12")
-    (pin "39_13")
-    (pin "39_14")
-    (pin "39_15")
-    (pin "39_16")
-    (pin "39_17")
-    (pin "39_18")
-    (pin "39_19")
     (pin "39_2")
-    (pin "39_20")
-    (pin "39_21")
     (pin "39_3")
     (pin "39_4")
