File: IR_EandR.kicad_sch (KiCad schematic)
At the start: 11 parts, among them J4 IR Emitter, J6 Conn_01x04, J8 IR Receiver, U6 LM293DRE4

Commit message: Annotations
Other:
- note added: "Pins 1 and 2 of this jumper allow the comparator and IR Receiver to be driven at 3.3V or 18V."
- note added: "Pins 3 and 4 allow me to connect the IR Emitter directly to the MCU or through a FET to VCC. This will depend on how much current is needed for the distances I plan to send the IR beam. By using a through-pin IR Diode, I also leave myself open to switch to a laser emitter if needed."
- note added: "R11 and R12 control the voltage threshold for the comparator. Their values are left undefined on the test board until more testing can be done on the IR Receiver."
- note added: "The IR Emitter resistor will control the current pulled through the emitter. Its value is undefined on the test board"
- note added: "The IR Receiver is a phototransistor, which allows a certain current based on how many photons are striking it. R9 is set so that current creates a readable voltage. It is left undefined on the test board."
- moved on the sheet: C5, J8, R10, R11, R12, R9, U6
