File: buzzer.kicad_sch (KiCad schematic)
At the start: 6 parts, among them J1 Conn_01x02, U4 UCC23313DWYR, U5 RD3L01BATTL1

Commit message: Annotations
Other:
- note added: "R5 is left undefined to allow for testing. To reduce power consumption, the highest resistance - without restricting the full oscillations of the piezzo - should be selected"
- note added: "R6 is left undefined to be decided later."
Changed lines of the file:
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@@
     (stroke (width 0) (type default))
+  )
+  (text "R5 is left undefined to allow\nfor testing. To reduce power\nconsumption, the highest\nresistance - without restricting\nthe full oscillations of the\npiezzo - should be selected"
+    (at 168.275 147.955 0)
+    (effects (font (size 1.27 1.27)) (justify left bottom))
   )
   (text "This design assumes that the PWM generator is capable of providing the Gate Driver operating current \nof 10mA"
@@
     (effects (font (size 1.27 1.27)) (justify left bottom))
   )
+  (text "R6 is left undefined to be\ndecided later." (at 116.84 114.3 0)
+    (effects (font (size 1.27 1.27)) (justify left bottom))
+  )
